Commit message: camera added

File: urdf/deliverybot.urdf.xacro (robot description, xacro)
@@ -129,35 +129,7 @@
     </inertial>
   </link>
-  <!-- <joint name="cam_left_joint" type="fixed">
-    <parent link="base_link"/>
-    <child link="cam_left_link"/>
-    <origin xyz="0.0362 -0.05 0.182" rpy="1.57 0 0.3"/>
-  </joint>
-  <link name="cam_left_link">
-    <visual>
-      <origin xyz="0 0 0.0" rpy="-1.57 0 -1.57"/>
-      <geometry>
-        <mesh filename="package://realsense2_description/meshes/d435.dae" scale="1 1 1"/>
-      </geometry>
-      <material name="dark"/>
-    </visual>
-  </link> -->
   <xacro:sensor_d435 name="cam_left" topics_ns="cam_left" parent="base_link" publish_pointcloud="true">
       <origin xyz="0.0302 -0.03 0.182" rpy="-1.57 0 0.3491" />
   </xacro:sensor_d435>
-  <!-- <joint name="cam_right_joint" type="fixed">
-    <parent link="base_link"/>
-    <child link="cam_right_link"/>
-    <origin xyz="0.0362 0.05 0.182" rpy="1.57 0 -0.3"/>
-  </joint>
-  <link name="cam_right_link">
-    <visual>
-      <origin xyz="0 0 0.0" rpy="-1.57 0 -1.57"/>
-      <geometry>
-        <mesh filename="package://realsense2_description/meshes/d435.dae" scale="1 1 1"/>
-      </geometry>
-      <material name="dark"/>
-    </visual>
-  </link> -->
   <xacro:sensor_d435 name="cam_right" topics_ns="cam_right" parent="base_link" publish_pointcloud="true">
       <origin xyz="0.0302 0.03 0.182" rpy="-1.57 0 -0.3491" />

Commit message: adjust FOV of realsense

File: urdf/deliverybot.urdf.xacro (robot description, xacro)
@@ -130,8 +130,8 @@
   </link>
   <xacro:sensor_d435 name="cam_left" topics_ns="cam_left" parent="base_link" publish_pointcloud="true">
-      <origin xyz="0.0302 -0.03 0.182" rpy="-1.57 0 0.3491" />
+      <origin xyz="0.0302 -0.03 0.182" rpy="-0.3491 1.57 0" />
   </xacro:sensor_d435>
   <xacro:sensor_d435 name="cam_right" topics_ns="cam_right" parent="base_link" publish_pointcloud="true">
-      <origin xyz="0.0302 0.03 0.182" rpy="-1.57 0 -0.3491" />
+      <origin xyz="0.0302 0.03 0.182" rpy="0.3491 1.57 0" />
   </xacro:sensor_d435>
 </robot>

Commit message: phase 1

File: urdf/deliverybot.urdf.xacro (robot description, xacro)
@@ -130,8 +130,10 @@
   </link>
   <xacro:sensor_d435 name="cam_left" topics_ns="cam_left" parent="base_link" publish_pointcloud="true">
-      <origin xyz="0.0302 -0.03 0.182" rpy="-0.3491 1.57 0" />
+      <origin xyz="0.0302 0.03 0.182" rpy="0 1.57 0" />
+      <!-- <origin xyz="0.0302 -0.1 0.182" rpy="-1.57 0 -1.57" /> -->
   </xacro:sensor_d435>
   <xacro:sensor_d435 name="cam_right" topics_ns="cam_right" parent="base_link" publish_pointcloud="true">
-      <origin xyz="0.0302 0.03 0.182" rpy="0.3491 1.57 0" />
+      <origin xyz="0.0302 -0.03 0.182" rpy="-0.3491 1.57 0" />
+      <!-- <origin xyz="0.0302 0.1 0.182" rpy="-1.57 0 -1.57" /> -->
   </xacro:sensor_d435>
 </robot>

Commit message: intrinsic done

File: urdf/deliverybot.urdf.xacro (robot description, xacro)
@@ -130,10 +130,8 @@
   </link>
   <xacro:sensor_d435 name="cam_left" topics_ns="cam_left" parent="base_link" publish_pointcloud="true">
-      <origin xyz="0.0302 0.03 0.182" rpy="0 1.57 0" />
-      <!-- <origin xyz="0.0302 -0.1 0.182" rpy="-1.57 0 -1.57" /> -->
+      <origin xyz="0.0302 0.03 0.182" rpy="-1.57 0 -2.3038" />
   </xacro:sensor_d435>
   <xacro:sensor_d435 name="cam_right" topics_ns="cam_right" parent="base_link" publish_pointcloud="true">
-      <origin xyz="0.0302 -0.03 0.182" rpy="-0.3491 1.57 0" />
-      <!-- <origin xyz="0.0302 0.1 0.182" rpy="-1.57 0 -1.57" /> -->
+      <origin xyz="0.0302 -0.03 0.182" rpy="-1.57 0 -0.8378" />
   </xacro:sensor_d435>
 </robot>
